Commit message: Corrected some paths

File: husky_description/urdf/custom_description.urdf.xacro (robot description, xacro)
@@ -25,5 +25,5 @@
   <xacro:arg name="ur5_enabled" default="$(optenv HUSKY_UR5_ENABLED false)" />
   <xacro:arg name="kinect_enabled" default="false" />
-  <xacro:include filename="$(find husky_cuarl)/husky_description/urdf/husky.urdf.xacro" />
+  <xacro:include filename="$(find husky_description)/urdf/husky.urdf.xacro" />
   <xacro:husky_robot />
   <!-- Insert customization below, sample provided: -->
@@ -31,5 +31,5 @@
     <visual>
       <geometry>
-        <mesh filename="package://husky_cuarl/husky_description/meshes/red_bowler.dae" />
+        <mesh filename="package://husky_description/meshes/red_bowler.dae" />
       </geometry>
     </visual>

File: husky_gazebo/urdf/custom_description.gazebo.xacro (robot description, xacro)
@@ -33,5 +33,5 @@
   </gazebo>
   <xacro:husky_robot_gazebo />
-  <xacro:include filename="$(find husky_custom_description)/urdf/custom_description.urdf.xacro" />
+  <xacro:include filename="$(find husky_description)/urdf/custom_description.urdf.xacro" />
   <!-- Insert customizations below: -->
 </robot>

Commit message: Successfully render hat

File: husky_description/urdf/custom_description.urdf.xacro (robot description, xacro)
@@ -25,24 +25,4 @@
   <xacro:arg name="ur5_enabled" default="$(optenv HUSKY_UR5_ENABLED false)" />
   <xacro:arg name="kinect_enabled" default="false" />
-  <xacro:include filename="$(find husky_description)/urdf/husky.urdf.xacro" />
-  <xacro:husky_robot />
   <!-- Insert customization below, sample provided: -->
-  <link name="bowler_link">
-    <visual>
-      <geometry>
-        <mesh filename="package://husky_description/meshes/red_bowler.dae" />
-      </geometry>
-    </visual>
-    <collision>
-      <origin xyz="0 0 0.07" rpy="0 0 0" />
-      <geometry>
-        <box size="0.32 0.25 0.14" rpy="0 0 0"/>
-      </geometry>
-    </collision>
-  </link>
-  <joint name="bowler_joint" type="fixed">
-    <parent link="top_plate_link" />
-    <child link="bowler_link" />
-    <origin xyz="0.1 -0.1 0" rpy="0 0 0.5" />
-  </joint>
 </robot>

File: husky_description/urdf/husky.urdf.xacro (robot description, xacro)
@@ -1,4 +1,3 @@
-<?xml version="1.0"?>
-<!--
+<?xml version="1.0"?> <!--
 Software License Agreement (BSD)
 \file      husky.urdf.xacro
@@ -35,5 +34,5 @@
   <xacro:property name="husky_rear_bumper_extend" value="$(optenv HUSKY_REAR_BUMPER_EXTEND 0)" />
   <xacro:arg name="robot_namespace" default="/" />
-  <xacro:arg name="urdf_extras" default="empty.urdf" />
+  <xacro:arg name="urdf_extras" default="$(find husky_description)/urdf/custom_description.urdf.xacro" />
   <!-- Included URDF/XACRO Files -->
   <xacro:include filename="$(find husky_description)/urdf/decorations.urdf.xacro" />
@@ -106,4 +105,26 @@
   <gazebo reference="imu_link">
   </gazebo>
+  <link name="bowler_link">
+    <visual>
+      <geometry>
+        <mesh filename="$(find husky_description)/meshes/red_bowler.dae" />
+      </geometry>
+    </visual>
+    <collision>
+      <origin xyz="0 0 0.07" rpy="0 0 0" />
+      <geometry>
+        <box size="0.32 0.25 0.14" rpy="0 0 0"/>
+      </geometry>
+    </collision>
+    <inertial>
+      <mass value="30"/>
+      <inertia ixx="0.4" ixy="0.0" ixz="0.0" iyy="0.4" iyz="0.0" izz="0.2"/>
+    </inertial>
+  </link>
+  <joint name="bowler_joint" type="fixed">
+    <parent link="top_plate_link" />
+    <child link="bowler_link" />
+    <origin xyz="0.02 0.2 0" rpy="0 0 0.5" />
+  </joint>
   <!-- Husky wheel macros -->
   <xacro:husky_wheel wheel_prefix="front_left">
@@ -193,5 +214,3 @@
     </plugin>
   </gazebo>
-  <!-- Optional custom includes. -->
-  <xacro:include filename="$(arg urdf_extras)" />
 </robot>
