Commit message: Add perfect COM for husky

File: husky_description/urdf/husky.urdf.xacro (robot description, xacro)
@@ -118,5 +118,5 @@
     </collision>
     <inertial>
-      <mass value="30"/>
+      <mass value="21.8"/>
       <inertia ixx="0.4" ixy="0.0" ixz="0.0" iyy="0.4" iyz="0.0" izz="0.2"/>
     </inertial>
@@ -125,5 +125,5 @@
     <parent link="top_plate_link" />
     <child link="bowler_link" />
-    <origin xyz="0.02 0.2 0" rpy="0 0 0.5" />
+    <origin xyz="-0.10 0.18 0" rpy="0 0 0.5" />
   </joint>
   <!-- Husky wheel macros -->
